Commit message: add table mesh in pybullet

File: pybullet_simulator/robots/franka/urdf/panda_arm_hand_realsense.urdf (robot description, URDF)
Before this commit: robot panda, 22 links, 21 joints
Links:
- added link table; collision mesh filename=meshes/visual/table.obj; visual mesh filename=meshes/visual/table.dae
Joints:
- added joint table_joint: type fixed, parent world, child table, origin xyz=0.0 0.0 -0.39 rpy=0.0 0.0 0.0
- joint realsense_optical_joint: origin xyz=0.0 0.015 0.0 rpy=-1.571 0, -1.571 -> xyz=0.0 0.015 0.0 rpy=-1.571 0 -1.571

Commit message: fix pybullet robot_description

File: pybullet_simulator/robots/franka/urdf/panda_arm_hand_realsense.urdf (robot description, URDF)
Before this commit: robot panda, 23 links, 22 joints
Links:
- link panda_hand: geometry collision mesh filename=package://pybullet_simulator/robots/franka/urdf/meshes/visu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; visual mesh filename=package://pybullet_simulator/robots/franka/urdf/meshes/visu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
- link panda_leftfinger: geometry collision mesh filename=package://pybullet_simulator/robots/franka/urdf/meshes/visu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; visual mesh filename=package://pybullet_simulator/robots/franka/urdf/meshes/visu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
- link panda_link0: geometry collision mesh filename=package://pybullet_simulator/robots/franka/urdf/meshes/visu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; visual mesh filename=package://pybullet_simulator/robots/franka/urdf/meshes/visu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
- link panda_link1: geometry collision mesh filename=package://pybullet_simulator/robots/franka/urdf/meshes/visu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; visual mesh filename=package://pybullet_simulator/robots/franka/urdf/meshes/visu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
- link panda_link2: geometry collision mesh filename=package://pybullet_simulator/robots/franka/urdf/meshes/visu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; visual mesh filename=package://pybullet_simulator/robots/franka/urdf/meshes/visu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
- link panda_link3: geometry collision mesh filename=package://pybullet_simulator/robots/franka/urdf/meshes/visu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; visual mesh filename=package://pybullet_simulator/robots/franka/urdf/meshes/visu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
- link panda_link4: geometry collision mesh filename=package://pybullet_simulator/robots/franka/urdf/meshes/visu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; visual mesh filename=package://pybullet_simulator/robots/franka/urdf/meshes/visu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
- link panda_link5: geometry collision mesh filename=package://pybullet_simulator/robots/franka/urdf/meshes/visu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; visual mesh filename=package://pybullet_simulator/robots/franka/urdf/meshes/visu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
- link panda_link6: geometry collision mesh filename=package://pybullet_simulator/robots/franka/urdf/meshes/visu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; visual mesh filename=package://pybullet_simulator/robots/franka/urdf/meshes/visu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
- link panda_link7: geometry collision mesh filename=package://pybullet_simulator/robots/franka/urdf/meshes/visu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; visual mesh filename=package://pybullet_simulator/robots/franka/urdf/meshes/visu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
- link panda_rightfinger: geometry collision mesh filename=package://pybullet_simulator/robots/franka/urdf/meshes/visu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; visual mesh filename=package://pybullet_simulator/robots/franka/urdf/meshes/visu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
- link realsense_link: geometry collision box size=0.02505 0.09 0.025; visual mesh filename=package://pybullet_simulator/robots/franka/urdf/meshes/visu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
- link table: geometry collision mesh filename=package://pybullet_simulator/robots/franka/urdf/meshes/visu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; visual mesh filename=package://pybullet_simulator/robots/franka/urdf/meshes/visu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

Commit message: prune

File: pybullet_simulator/robots/franka/urdf/panda_arm_hand_realsense.urdf (robot description, URDF)
Before this commit: robot panda, 23 links, 22 joints
Links:
- link panda_hand: geometry collision mesh filename=package://../drivers/franka_ros/franka_description/meshes/v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; visual mesh filename=package://../drivers/franka_ros/franka_description/meshes/v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
- link panda_leftfinger: geometry collision mesh filename=package://../ocrtoc_task/config/meshes/finger.dae; visual mesh filename=package://../ocrtoc_task/config/meshes/finger.dae
- link panda_link0: geometry collision mesh filename=package://../drivers/franka_ros/franka_description/meshes/v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; visual mesh filename=package://../drivers/franka_ros/franka_description/meshes/v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
- link panda_link1: geometry collision mesh filename=package://../drivers/franka_ros/franka_description/meshes/v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; visual mesh filename=package://../drivers/franka_ros/franka_description/meshes/v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
- link panda_link2: geometry collision mesh filename=package://../drivers/franka_ros/franka_description/meshes/v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; visual mesh filename=package://../drivers/franka_ros/franka_description/meshes/v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
- link panda_link3: geometry collision mesh filename=package://../drivers/franka_ros/franka_description/meshes/v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; visual mesh filename=package://../drivers/franka_ros/franka_description/meshes/v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
- link panda_link4: geometry collision mesh filename=package://../drivers/franka_ros/franka_description/meshes/v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; visual mesh filename=package://../drivers/franka_ros/franka_description/meshes/v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
- link panda_link5: geometry collision mesh filename=package://../drivers/franka_ros/franka_description/meshes/v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; visual mesh filename=package://../drivers/franka_ros/franka_description/meshes/v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
- link panda_link6: geometry collision mesh filename=package://../drivers/franka_ros/franka_description/meshes/v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; visual mesh filename=package://../drivers/franka_ros/franka_description/meshes/v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
- link panda_link7: geometry collision mesh filename=package://../drivers/franka_ros/franka_description/meshes/v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; visual mesh filename=package://../drivers/franka_ros/franka_description/meshes/v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
- link panda_rightfinger: geometry collision mesh filename=package://../ocrtoc_task/config/meshes/finger.dae; visual mesh filename=package://../ocrtoc_task/config/meshes/finger.dae
- link realsense_link: geometry collision box size=0.02505 0.09 0.025; visual mesh filename=package://../drivers/realsense-ros/realsense2_description/m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
- link table: geometry collision mesh filename=package://../ocrtoc_task/config/meshes/table/collision/tabl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; visual mesh filename=package://../ocrtoc_task/config/meshes/table/visual/table.d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
